Commit message: recreated pr2.urdf from xacro file

File: share/data/pr2_model/pr2.urdf (robot description, URDF)
Before this commit: robot pr2, 95 links, 94 joints
Links:
- removed link narrow_stereo_gazebo_l_stereo_camera_frame
- removed link narrow_stereo_gazebo_l_stereo_camera_optical_frame
- removed link narrow_stereo_gazebo_r_stereo_camera_frame
- removed link narrow_stereo_gazebo_r_stereo_camera_optical_frame
- removed link wide_stereo_gazebo_l_stereo_camera_frame
- removed link wide_stereo_gazebo_l_stereo_camera_optical_frame
- removed link wide_stereo_gazebo_r_stereo_camera_frame
- removed link wide_stereo_gazebo_r_stereo_camera_optical_frame
- added link narrow_stereo_l_stereo_camera_frame, mass 0.01
- added link narrow_stereo_l_stereo_camera_optical_frame
- added link narrow_stereo_r_stereo_camera_frame, mass 0.01
- added link narrow_stereo_r_stereo_camera_optical_frame
- added link wide_stereo_l_stereo_camera_frame, mass 0.01
- added link wide_stereo_l_stereo_camera_optical_frame
- added link wide_stereo_r_stereo_camera_frame, mass 0.01
- added link wide_stereo_r_stereo_camera_optical_frame
Joints:
- removed joint narrow_stereo_gazebo_l_stereo_camera_frame_joint
- removed joint narrow_stereo_gazebo_l_stereo_camera_optical_frame_joint
- removed joint narrow_stereo_gazebo_r_stereo_camera_frame_joint
- removed joint narrow_stereo_gazebo_r_stereo_camera_optical_frame_joint
- removed joint wide_stereo_gazebo_l_stereo_camera_frame_joint
- removed joint wide_stereo_gazebo_l_stereo_camera_optical_frame_joint
- removed joint wide_stereo_gazebo_r_stereo_camera_frame_joint
- removed joint wide_stereo_gazebo_r_stereo_camera_optical_frame_joint
- added joint narrow_stereo_l_stereo_camera_frame_joint: type fixed, parent narrow_stereo_link, child narrow_stereo_l_stereo_camera_frame, origin xyz=0 0 0 rpy=0 0 0
- added joint narrow_stereo_l_stereo_camera_optical_frame_joint: type fixed, parent narrow_stereo_l_stereo_camera_frame, child narrow_stereo_l_stereo_camera_optical_frame, origin xyz=0 0 0 rpy=-1.57079632679 0.0 -1.57079632679
- added joint narrow_stereo_r_stereo_camera_frame_joint: type fixed, parent narrow_stereo_l_stereo_camera_frame, child narrow_stereo_r_stereo_camera_frame, origin xyz=0.0 -0.09 0.0 rpy=0.0 0.0 0.0
- added joint narrow_stereo_r_stereo_camera_optical_frame_joint: type fixed, parent narrow_stereo_r_stereo_camera_frame, child narrow_stereo_r_stereo_camera_optical_frame, origin xyz=0 0 0 rpy=-1.57079632679 0.0 -1.57079632679
- added joint wide_stereo_l_stereo_camera_frame_joint: type fixed, parent wide_stereo_link, child wide_stereo_l_stereo_camera_frame, origin xyz=0 0 0 rpy=0 0 0
- added joint wide_stereo_l_stereo_camera_optical_frame_joint: type fixed, parent wide_stereo_l_stereo_camera_frame, child wide_stereo_l_stereo_camera_optical_frame, origin xyz=0 0 0 rpy=-1.57079632679 0.0 -1.57079632679
- added joint wide_stereo_r_stereo_camera_frame_joint: type fixed, parent wide_stereo_l_stereo_camera_frame, child wide_stereo_r_stereo_camera_frame, origin xyz=0.0 -0.09 0.0 rpy=0.0 0.0 0.0
- added joint wide_stereo_r_stereo_camera_optical_frame_joint: type fixed, parent wide_stereo_r_stereo_camera_frame, child wide_stereo_r_stereo_camera_optical_frame, origin xyz=0 0 0 rpy=-1.57079632679 0.0 -1.57079632679
- joint bl_caster_l_wheel_joint: limit effort=100 velocity=100 -> effort=7 velocity=15
- joint bl_caster_r_wheel_joint: limit effort=100 velocity=100 -> effort=7 velocity=15
- joint bl_caster_rotation_joint: limit effort=100 velocity=100 -> effort=6.5 velocity=10
- joint br_caster_l_wheel_joint: limit effort=100 velocity=100 -> effort=7 velocity=15
- joint br_caster_r_wheel_joint: limit effort=100 velocity=100 -> effort=7 velocity=15
- joint br_caster_rotation_joint: limit effort=100 velocity=100 -> effort=6.5 velocity=10
- joint fl_caster_l_wheel_joint: limit effort=100 velocity=100 -> effort=7 velocity=15
- joint fl_caster_r_wheel_joint: limit effort=100 velocity=100 -> effort=7 velocity=15
- joint fl_caster_rotation_joint: limit effort=100 velocity=100 -> effort=6.5 velocity=10
- joint fr_caster_l_wheel_joint: limit effort=100 velocity=100 -> effort=7 velocity=15
- joint fr_caster_r_wheel_joint: limit effort=100 velocity=100 -> effort=7 velocity=15
- joint fr_caster_rotation_joint: limit effort=100 velocity=100 -> effort=6.5 velocity=10
- joint head_mount_kinect_ir_optical_frame_joint: origin xyz=0.0            0.0         0.0 rpy=-1.57079632679 0.0 -1.57079632679 -> xyz=0.0            0.01         0.0 rpy=-1.57079632679 0.0 -1.57079632679
